Commit message: Update robot.urdf to full 6-DOF Thor arm model

File: robot.urdf (robot description, URDF)
Before this commit: robot thor_arm, 2 links, 1 joints
Links:
- added link link_2; visual cylinder length=0.25 radius=0.04
- added link link_3; visual cylinder length=0.2 radius=0.035
- added link link_4; visual cylinder length=0.15 radius=0.03
- added link link_5; visual cylinder length=0.1 radius=0.025
- added link link_6; visual cylinder length=0.05 radius=0.02
- link link_1: geometry visual cylinder length=0.15 radius=0.05
Joints:
- added joint joint_2: type revolute, parent link_1, child link_2, origin xyz=0 0 0.15 rpy=0 1.57 0, axis 0 1 0, limit lower=-2.0 upper=2.0 effort=10.0 velocity=1.0
- added joint joint_3: type revolute, parent link_2, child link_3, origin xyz=0 0 0.25 rpy=0 0 0, axis 0 0 1, limit lower=-2.0 upper=2.0 effort=10.0 velocity=1.0
- added joint joint_4: type revolute, parent link_3, child link_4, origin xyz=0 0 0.2 rpy=0 0 0, axis 1 0 0, limit lower=-3.14 upper=3.14 effort=5.0 velocity=1.5
- added joint joint_5: type revolute, parent link_4, child link_5, origin xyz=0 0 0.15 rpy=0 0 0, axis 0 1 0, limit lower=-2.0 upper=2.0 effort=5.0 velocity=1.5
- added joint joint_6: type revolute, parent link_5, child link_6, origin xyz=0 0 0.1 rpy=0 0 0, axis 0 0 1, limit lower=-3.14 upper=3.14 effort=5.0 velocity=2.0
- joint joint_1: origin xyz=0 0 0.05 rpy=0 0 0 -> xyz=0 0 0.1 rpy=0 0 0
